File: SlopesMain/SlopeMain1.kicad_sch (KiCad schematic)
At the start: 64 parts, among them J1 Synth_power_2x5, Q1 2N3906, Q2 2N3906, Q3 2N3904, Q4 2N3904, U1 TL072, U2 TL072, U3 TL074, U4 TLC3702, U5 TL072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

Commit message: Updated Schematic
Other:
- title: (none) -> Kosmo Slopes
Changed lines of the file:
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@@
 (kicad_sch (version 20230121) (generator eeschema)
   (paper "A4")
+  (title_block
+    (title "Kosmo Slopes")
+    (date "2023-03-18")
+  )
   (junction (at 102.87 189.23) (diameter 0) (color 0 0 0 0)
   )
