File: SlopesMain/SlopeMain2.kicad_sch (KiCad schematic)
At the start: 29 parts, among them J2 Conn_01x12, SW1 SW_SPDT, U5 TL072, U6 TL072

Commit message: Updated Schematic
Other:
- title: (none) -> Kosmo Slopes
Changed lines of the file:
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@@
 (kicad_sch (version 20230121) (generator eeschema)
   (paper "A4")
+  (title_block
+    (title "Kosmo Slopes")
+    (date "2023-03-18")
+  )
   (junction (at 232.41 77.47) (diameter 0) (color 0 0 0 0)
   )
