File: SlopesMain/SlopesMain.kicad_sch (KiCad schematic)
At the start: 0 parts

Commit message: Updated Schematic
Other:
- title: (none) -> Kosmo Slopes
Changed lines of the file:
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@@
 (kicad_sch (version 20230121) (generator eeschema)
   (paper "A4")
+  (title_block
+    (title "Kosmo Slopes")
+    (date "2023-03-18")
+  )
   (sheet (at 130.175 73.025) (size 22.225 35.56) (fields_autoplaced)
     (stroke (width 0.1524) (type solid))
